File: PCB/ratless65.kicad_pcb (KiCad board)
At the start: 2 copper layers, 132 parts, among them U1 ProMicro, U2 ProMicro

Commit message: Started wiring to the MCUs + Added TRRS jacks + Lots...
Parts:
- added J1: MJ-4PP-9, MJ-4PP-9:MJ-4PP-9, F.Cu at (183.4, 72.8)
- added J2: MJ-4PP-9, MJ-4PP-9:MJ-4PP-9, F.Cu at (158.0, 73.0)
- D1, D10, D11, D12, D13, D14, D15, D16, D17, D18, D19, D2, D20, D21, D22, D23, D24, D25, D26, D27, D28, D29, D3, D30, D31, D32, D33, D34, D35, D36, D37, D38, D39, D4, D40, D41, D42, D43, D44, D45, D46, D47, D48, D49, D5, D50, D51, D52, D53, D54, D55, D56, D57, D58, D59, D6, D60, D61, D62, D63, D64, D65, D7, D8, D9: moved to B.Cu
- MX41, MX53: footprint PCM_marbastlib-mx:SW_MX_1u -> PCM_marbastlib-mx:SW_MX_1.5u
- moved MX54 387.6 mm to (42.9, 117.5)
- moved MX55 366.4 mm to (61.9, 117.5)
- moved MX42 356.7 mm to (38.1, 98.4)
- moved MX56 345.4 mm to (81.0, 115.9)
- moved MX43 332.4 mm to (61.9, 98.4)
- moved D1 326.6 mm to (41.3, 45.2), turned to 90 degrees
- moved MX57 325.0 mm to (100.0, 114.3)
- moved MX45 318.6 mm to (100.0, 95.2)
- moved MX44 313.6 mm to (81.0, 96.8)
- moved MX59 312.5 mm to (142.9, 117.5)
- moved MX58 305.4 mm to (119.1, 115.9)
- moved MX46 297.0 mm to (119.1, 96.8)
- moved D42 295.1 mm to (41.3, 102.3), turned to 90 degrees
- moved D54 294.1 mm to (46.0, 121.4), turned to 90 degrees
- moved D15 286.5 mm to (41.3, 64.4), turned to 90 degrees
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Connections:
- net Net-(D21-K) renamed ROW6
- net Net-(D35-K) renamed ROW7
- net Net-(D48-K) renamed ROW8
- net Net-(D60-K) renamed ROW9
- net Net-(MX1-Pad1) renamed COL0
- net Net-(MX10-Pad1) renamed COL9
- net Net-(MX11-Pad1) renamed COL10
- net Net-(MX12-Pad1) renamed COL11
- net Net-(MX13-Pad1) renamed COL12
- net Net-(MX14-Pad1) renamed COL13
- net Net-(MX16-Pad1) renamed COL1
- net Net-(MX17-Pad1) renamed COL2
- net Net-(MX18-Pad1) renamed COL3
- net Net-(MX19-Pad1) renamed COL4
- net Net-(MX20-Pad1) renamed COL5
- net Net-(MX21-Pad1) renamed COL6
- net Net-(MX22-Pad1) renamed COL7
- net Net-(MX23-Pad1) renamed COL8
- D1 pad 1: Net-(D1-K) -> ROW0
- D10 pad 1: unconnected-(D10-K-Pad1) -> ROW5
- D11 pad 1: unconnected-(D11-K-Pad1) -> ROW5
- D12 pad 1: unconnected-(D12-K-Pad1) -> ROW5
- D13 pad 1: unconnected-(D13-K-Pad1) -> ROW5
- D14 pad 1: unconnected-(D14-K-Pad1) -> ROW5
- D15 pad 1: Net-(D15-K) -> ROW1
- D16 pad 1: Net-(D15-K) -> ROW1
- D17 pad 1: Net-(D15-K) -> ROW1
- D18 pad 1: Net-(D15-K) -> ROW1
- D19 pad 1: Net-(D15-K) -> ROW1
- D2 pad 1: Net-(D1-K) -> ROW0
- D20 pad 1: Net-(D15-K) -> ROW1
- D29 pad 1: Net-(D29-K) -> ROW2
- D3 pad 1: Net-(D1-K) -> ROW0
- D30 pad 1: Net-(D29-K) -> ROW2
- D31 pad 1: Net-(D29-K) -> ROW2
- D32 pad 1: Net-(D29-K) -> ROW2
- D33 pad 1: Net-(D29-K) -> ROW2
- D34 pad 1: Net-(D29-K) -> ROW2
- D4 pad 1: Net-(D1-K) -> ROW0
- D42 pad 1: Net-(D42-K) -> ROW3
- D43 pad 1: Net-(D42-K) -> ROW3
- D44 pad 1: Net-(D42-K) -> ROW3
- D45 pad 1: Net-(D42-K) -> ROW3
- D46 pad 1: Net-(D42-K) -> ROW3
- D47 pad 1: Net-(D42-K) -> ROW3
- D5 pad 1: Net-(D1-K) -> ROW0
- D54 pad 1: Net-(D54-K) -> ROW4
- D55 pad 1: Net-(D54-K) -> ROW4
- D56 pad 1: Net-(D54-K) -> ROW4
- D57 pad 1: Net-(D54-K) -> ROW4
- D58 pad 1: Net-(D54-K) -> ROW4
- D59 pad 1: Net-(D54-K) -> ROW4
- D6 pad 1: Net-(D1-K) -> ROW0
- D7 pad 1: unconnected-(D7-K-Pad1) -> ROW5
- D8 pad 1: unconnected-(D8-K-Pad1) -> ROW5
- D9 pad 1: unconnected-(D9-K-Pad1) -> ROW5
- U1 pad 16: unconnected-(U1-VCC-Pad16) -> VCC
- U1 pad 2: unconnected-(U1-D2-RX-Pad2) -> dataU1
- U1 pad 3: unconnected-(U1-GND-Pad3) -> GND
- U1 pad 4: unconnected-(U1-GND-Pad4) -> GND
- U2 pad 16: unconnected-(U2-VCC-Pad16) -> VCC
- U2 pad 2: unconnected-(U2-D2-RX-Pad2) -> dataU2
- U2 pad 3: unconnected-(U2-GND-Pad3) -> GND
- U2 pad 4: unconnected-(U2-GND-Pad4) -> GND
- U2 pad 5: unconnected-(U2-D1-Pad5) -> ROW0
- U2 pad 6: unconnected-(U2-D0-Pad6) -> ROW1
- U2 pad 7: unconnected-(U2-D4-Pad7) -> ROW2
- U2 pad 8: unconnected-(U2-C6-Pad8) -> ROW3
- U2 pad 9: unconnected-(U2-D7-Pad9) -> ROW4
Routing:
- net ROW4: track 0.00 -> 175.1 mm
- net ROW3: track 0.00 -> 161.0 mm
- net ROW2: track 0.00 -> 144.4 mm
- net ROW6: track 0.00 -> 138.4 mm
- net ROW5: track 0.00 -> 138.4 mm
- net ROW1: track 0.00 -> 127.7 mm
- net ROW0: track 0.00 -> 111.6 mm
- net ROW9: track 0.00 -> 102.7 mm
- net ROW8: track 0.00 -> 102.6 mm
- net ROW7: track 0.00 -> 97.9 mm
- net COL11: track 0.00 -> 80.7 mm
- net COL6: track 0.00 -> 79.2 mm
- net COL0: track 0.00 -> 78.3 mm
- net COL5: track 0.00 -> 78.2 mm
- net GND: track 0.00 -> 77.4 mm
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
Commit message: Finished PCB, need to add resistors for I2C
Parts:
- added REF**: mousebites 2mm, PCM_marbastlib-various:mousebites_2.5mm, F.Cu at (178.6, 31.8)
- added REF**: mousebites 2mm, PCM_marbastlib-various:mousebites_2.5mm, F.Cu at (162.7, 31.8)
- added REF**: mousebites 2mm, PCM_marbastlib-various:mousebites_2.5mm, F.Cu at (38.1, 126.2)
- added REF**: mousebites 2mm, PCM_marbastlib-various:mousebites_2.5mm, F.Cu at (162.7, 126.2)
- added REF**: mousebites 2mm, PCM_marbastlib-various:mousebites_2.5mm, F.Cu at (28.6, 32.5)
- added REF**: mousebites 2mm, PCM_marbastlib-various:mousebites_2.5mm, F.Cu at (303.2, 126.2)
- added REF**: mousebites 2mm, PCM_marbastlib-various:mousebites_2.5mm, F.Cu at (178.6, 126.2)
- added REF**: mousebites 2mm, PCM_marbastlib-various:mousebites_2.5mm, F.Cu at (346.1, 32.5)
Connections:
- U1 pad 10: unconnected-(U1-E6-Pad10) -> COL11
- U1 pad 11: unconnected-(U1-B4-Pad11) -> COL12
- U1 pad 12: unconnected-(U1-B5-Pad12) -> COL13
- U1 pad 17: unconnected-(U1-F4-Pad17) -> ROW5
- U1 pad 18: unconnected-(U1-F5-Pad18) -> ROW6
- U1 pad 19: unconnected-(U1-F6-Pad19) -> ROW7
- U1 pad 20: unconnected-(U1-F7-Pad20) -> ROW8
- U1 pad 21: unconnected-(U1-B1-Pad21) -> ROW9
- U1 pad 5: unconnected-(U1-D1-Pad5) -> COL9
- U1 pad 6: unconnected-(U1-D0-Pad6) -> COL8
- U1 pad 7: unconnected-(U1-D4-Pad7) -> COL7
- U1 pad 8: unconnected-(U1-C6-Pad8) -> COL6
- U1 pad 9: unconnected-(U1-D7-Pad9) -> COL10
- U2 pad 17: unconnected-(U2-F4-Pad17) -> COL0
- U2 pad 18: unconnected-(U2-F5-Pad18) -> COL1
- U2 pad 19: unconnected-(U2-F6-Pad19) -> COL2
- U2 pad 20: unconnected-(U2-F7-Pad20) -> COL3
- U2 pad 21: unconnected-(U2-B1-Pad21) -> COL4
- U2 pad 22: unconnected-(U2-B3-Pad22) -> COL5
Routing:
- net COL13: track 19.0 -> 302.7 mm
- net COL12: track 41.3 -> 291.3 mm
- net COL11: track 80.7 -> 272.6 mm
- net COL10: track 76.2 -> 248.6 mm
- net COL0: track 78.3 -> 228.3 mm
- net COL1: track 76.2 -> 203.3 mm
- net COL2: track 76.2 -> 185.9 mm
- net COL9: track 76.2 -> 173.3 mm
- net COL3: track 76.2 -> 167.9 mm
- net ROW9: track 102.7 -> 183.1 mm
- net COL8: track 76.2 -> 155.0 mm
- net ROW7: track 97.9 -> 169.4 mm
- net COL4: track 76.2 -> 144.6 mm
- net ROW8: track 102.6 -> 166.4 mm
- net COL7: track 76.2 -> 135.4 mm
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- added copper zone on B.Cu, net (none)
- added copper zone on F.Cu, net (none)
Other:
- board outline added: 326.2 x 116.8 mm

Commit message: I have no clue what changed but just want everything synced
Parts:
- removed the REF** at (178.6, 31.8)
- removed the REF** at (162.7, 31.8)
- removed the REF** at (38.1, 126.2)
- removed the REF** at (162.7, 126.2)
- removed the REF** at (28.6, 32.5)
- removed the REF** at (303.2, 126.2)
- removed the REF** at (178.6, 126.2)
- removed the REF** at (346.1, 32.5)
- added R1: 4.7k, PCM_Resistor_SMD_AKL:R_1206_3216Metric, F.Cu at (161.1, 59.4)
- added R2: 4.7k, PCM_Resistor_SMD_AKL:R_1206_3216Metric, F.Cu at (188.1, 57.9)
- added REF**: mousebites 2mm, PCM_marbastlib-various:mousebites_2mm, F.Cu at (178.6, 31.8)
- added REF**: mousebites 2mm, PCM_marbastlib-various:mousebites_2mm, F.Cu at (162.7, 31.8)
- added REF**: mousebites 2mm, PCM_marbastlib-various:mousebites_2mm, F.Cu at (162.7, 126.2)
- added REF**: mousebites 2mm, PCM_marbastlib-various:mousebites_2mm, F.Cu at (346.1, 32.5)
- added REF**: mousebites 2mm, PCM_marbastlib-various:mousebites_2mm, F.Cu at (28.6, 32.5)
- added REF**: mousebites 2mm, PCM_marbastlib-various:mousebites_2mm, F.Cu at (303.2, 126.2)
- added REF**: mousebites 2mm, PCM_marbastlib-various:mousebites_2mm, F.Cu at (178.6, 126.2)
- added REF**: mousebites 2mm, PCM_marbastlib-various:mousebites_2mm, F.Cu at (38.1, 126.2)
Connections:
- U1 pad 24: unconnected-(U1-B6-Pad24) -> Net-(U1-B6)
- U1 pad 5: COL9 -> COL6
- U1 pad 6: COL8 -> COL7
- U1 pad 7: COL7 -> COL8
- U1 pad 8: COL6 -> COL9
- U2 pad 10: unconnected-(U2-E6-Pad10) -> COL5
- U2 pad 17: COL0 -> ROW0
- U2 pad 18: COL1 -> ROW1
- U2 pad 19: COL2 -> ROW2
- U2 pad 20: COL3 -> ROW3
- U2 pad 21: COL4 -> ROW4
- U2 pad 22: COL5 -> unconnected-(U2-B3-Pad22)
- U2 pad 24: unconnected-(U2-B6-Pad24) -> Net-(U2-B6)
- U2 pad 5: ROW0 -> COL0
- U2 pad 6: ROW1 -> COL1
- U2 pad 7: ROW2 -> COL2
- U2 pad 8: ROW3 -> COL3
- U2 pad 9: ROW4 -> COL4
Routing:
- net COL8: track 155.0 -> 210.1 mm
- net COL9: track 173.3 -> 227.4 mm
- net COL7: track 135.4 -> 188.2 mm
- net COL1: track 203.3 -> 247.5 mm
- net COL0: track 228.3 -> 271.8 mm
- net COL5: track 126.3 -> 94.3 mm
- net ROW1: track 127.7 -> 158.5 mm
- net COL3: track 167.9 -> 148.6 mm
- net GND: track 77.4 -> 96.1 mm
- net COL6: track 104.8 -> 122.9 mm
- net COL2: track 185.9 -> 168.3 mm
- net ROW2: track 144.4 -> 159.8 mm
- net COL13: track 302.7 -> 290.2 mm
- net COL12: track 291.3 -> 280.0 mm
- net COL4: track 144.6 -> 133.3 mm
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Other:
- board size 326.2 x 116.8 mm -> 326.2 x 115.9 mm
